File: pcb/Vestax PDX-2000 Phono Preamp.kicad_sch (KiCad schematic)
At the start: 57 parts, among them J4 OUT_JU03_PU01, U1 LM2940CT-12_NOPB, U2 LM2990SX-12, U3 LM4562

Commit message: Added C2 value to schematic.
Parts:
- C2: value C -> 33u
Changed lines of the file:
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@@
       (effects (font (size 1.27 1.27)) (justify left))
     )
-    (property "Value" "C" (id 1) (at 73.66 87.6299 0)
+    (property "Value" "33u" (id 1) (at 73.66 87.6299 0)
       (effects (font (size 1.27 1.27)) (justify left))
     )
@@
     )
     (path "/2398130b-3ced-46f7-bd20-68a8905f6282"
-      (reference "C2") (unit 1) (value "C") (footprint "Capacitor_THT:CP_Radial_Tantal_D9.0mm_P5.00mm")
+      (reference "C2") (unit 1) (value "33u") (footprint "Capacitor_THT:CP_Radial_Tantal_D9.0mm_P5.00mm")
     )
     (path "/29b53c85-2641-4f1c-8ad3-b4972ce9fb90"
